File: pcb/audio_dsp_board/audio.kicad_sch (KiCad schematic)
At the start: 17 parts, among them J1 AudioJack4, J2 AudioJack4, U2 SGTL5000XNLA3

Commit message: Schematic capture, placement, routing complete
Sending board to JLCPCB for manufacturing and assembly.
Parts:
- C14, C15: footprint Capacitor_SMD:C_0402_1005Metric -> Capacitor_Tantalum_SMD:CP_EIA-3528-12_Kemet-T
- FB1: footprint (none) -> Diode_SMD:D_0603_1608Metric
- J1, J2: footprint (none) -> Connector_Audio:Jack_3.5mm_PJ320D_Horizontal
- R3: footprint (none) -> Resistor_SMD:R_0402_1005Metric
Changed lines of the file:
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@@
 			)
 		)
-		(property "Footprint" "Capacitor_SMD:C_0402_1005Metric"
+		(property "Footprint" "Capacitor_Tantalum_SMD:CP_EIA-3528-12_Kemet-T"
 			(at 123.19 113.9952 0)
 			(effects
@@
 			)
 		)
-		(property "Footprint" ""
+		(property "Footprint" "Connector_Audio:Jack_3.5mm_PJ320D_Horizontal"
 			(at 246.38 72.39 0)
 			(effects
@@
 			)
 		)
-		(property "Footprint" ""
+		(property "Footprint" "Resistor_SMD:R_0402_1005Metric"
 			(at 205.74 114.808 90)
 			(effects
@@
 			)
 		)
-		(property "Footprint" "Capacitor_SMD:C_0402_1005Metric"
+		(property "Footprint" "Capacitor_Tantalum_SMD:CP_EIA-3528-12_Kemet-T"
 			(at 123.19 122.8852 0)
 			(effects
@@
 			)
 		)
-		(property "Footprint" ""
+		(property "Footprint" "Diode_SMD:D_0603_1608Metric"
 			(at 147.32 69.088 90)
 			(effects
@@
 			)
 		)
-		(property "Footprint" ""
+		(property "Footprint" "Connector_Audio:Jack_3.5mm_PJ320D_Horizontal"
 			(at 246.38 106.68 0)
 			(effects
