File: pcb/audio_dsp_board/mcu.kicad_sch (KiCad schematic)
At the start: 27 parts, among them J3 Conn_01x04_Pin, SW1 SW_Push, SW2 SW_SPDT, SW3 SW_SPDT, U1 STM32F405RGTx, Y1 16MHz

Commit message: Schematic capture, placement, routing complete
Sending board to JLCPCB for manufacturing and assembly.
Parts:
- added C30: 100n, Capacitor_SMD:C_0402_1005Metric, symbol Device:C
- C2: footprint Capacitor_SMD:C_0402_1005Metric -> Capacitor_SMD:C_0603_1608Metric
- D2, D3: footprint (none) -> Diode_SMD:D_0603_1608Metric
- J3: footprint (none) -> Connector_PinHeader_2.54mm:PinHeader_1x04_P2.54mm_Vertical
- R1, R10, R11, R2, R6, R7, R8: footprint (none) -> Resistor_SMD:R_0402_1005Metric
- RV1: footprint (none) -> AAA:TRIM_3362P-1-103LF
- SW1: footprint (none) -> AAA:EL23520JLFS
- SW2, SW3: footprint (none) -> Button_Switch_SMD:SW_SPDT_PCM12
- Y1: footprint (none) -> Crystal:Crystal_SMD_3225-4Pin_3.2x2.5mm
Connections:
- net +3V3: now also C30.1
- net GND: now also SW1.2, C30.2; no longer SW1.1
- net NRST: now also SW1.1; no longer SW1.2
Other:
- moved on the sheet: C16, C17, C2, C3, C5, C6, C8, C9, D3, J3, R11, R2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
